File: VoltageProcessor.kicad_pcb (KiCad board)
At the start: 2 copper layers, 25.4 x 100 mm, 29 parts, among them J1 PJ301M-12, J2 PJ301M-12, J3 Eurorack power, J4 PJ301M-12, J5 PJ301M-12, U1 TL074

Commit message: Connected input CV jack's switch to GND instead of NC Add schematic picture
Connections:
- J1 pad 2: unconnected-(J1-Pad2) -> GND
- J2 pad 2: unconnected-(J2-Pad2) -> GND
